File: 3D-Printer/Cooler-7805-nano.brd (EAGLE design)
At the start: 100 x 75 mm, 40 parts, among them IC1 L293D, IC3 7805T, IC4 REG1117

Commit message: correct meters
meters and serial needed reversed.
Parts:
- removed U$1: ARDUINOMICRO, adafruit:ARDUINOMICRO
- added LCD_SCL, LCD_SDA: WIREPAD3,81/1,4, wirepad:3,81/1,4
- added U$2: NANO, Arduino-clone:NANO
- moved SET_CHAS 29.6 mm to (43.2, 71.1)
- moved SET_BED 21.6 mm to (38.1, 71.1)
- moved R7 3.81 mm to (29.2, 21.6)
- moved R9 2.54 mm to (25.4, 24.1)
- moved R10 2.54 mm to (15.2, 30.5)
- moved R8 2.54 mm to (15.2, 26.7)
- moved D1 2.54 mm to (21.6, 11.4)
Connections:
- removed net N$23: SET_BED.1, U$1.P$29
- removed net N$24: SET_CHAS.1, U$1.P$28
- new net N$18: SET_BED.1, U$2.A6
- new net N$20: R7.1, R8.2, U$2.A3
- new net N$44: LCD_SDA.1, U$2.A4
- new net N$45: LCD_SCL.1, U$2.A5
- net +3V3: now also U$2.3.3V, U$2.AREF; no longer U$1.P$32, U$1.P$33
- net +5V: now also U$2.5V; no longer U$1.P$23
- net GND: now also U$2.GND, U$2.GND1; no longer U$1.P$12, U$1.P$21
- net N$14: now also U$2.D2; no longer U$1.P$11
- net N$19: now also U$2.D3; no longer U$1.P$10
- net N$25: now also R10.2, R9.1, U$2.A2; no longer R7.1, R8.2, U$1.P$26
- net N$26: now also SET_CHAS.1, U$2.A7; no longer R10.2, R9.1, U$1.P$27
- net N$4: now also U$2.A0; no longer U$1.P$31
- net N$6: now also U$2.A1; no longer U$1.P$30
Routing:
- net N$20: track 0.00 -> 43.2 mm
- net N$26: track 31.8 -> 0.00 mm
- net N$24: track 14.8 -> 2.54 mm
- net N$45: track 0.00 -> 10.2 mm
- net N$6: track 39.5 -> 48.4 mm
- net GND: track 35.7 -> 44.5 mm
- net N$23: track 13.2 -> 5.08 mm
- net N$44: track 0.00 -> 8.15 mm
- net N$25: track 34.4 -> 40.4 mm
- net N$7: track 23.7 -> 29.0 mm
- net +12V: track 139.6 -> 144.7 mm
- net +3V3: track 37.2 -> 40.9 mm
- net N$8: track 9.19 -> 11.7 mm
- net N$43: track 0.00 -> 2.54 mm
- net N$41: track 0.00 -> 2.54 mm
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
Commit message: Added bounce capacitor
Corrected bounce on switch
Parts:
- added CY6: (no value), resistor:YC7B5
- moved IC4 82.7 mm to (3.81, 61.0)
- moved SET_CHAS 41.9 mm to (33.0, 30.5)
- moved SET_BED 35.9 mm to (33.0, 35.6)
- moved R3 5.08 mm to (74.9, 63.5)
- moved T1 5.08 mm to (77.5, 55.9)
- moved R4 2.54 mm to (77.5, 49.5)
Connections:
- net +5V: now also CY6.2
- net N$19: now also CY6.1
Routing:
- net N$19: track 22.1 -> 27.0 mm
- net +5V: track 227.0 -> 229.8 mm
- net N$5: track 14.5 -> 15.7 mm
- net N$14: track 31.8 -> 32.7 mm
